File: hardware/main-board/main-board.kicad_pcb (KiCad board)
At the start: 4 copper layers, 60 x 50 mm, 154 parts, among them J1 USB-C, J2 BATTERY 1S Li-ion (protected), J3 EXT BUTTON, J4 SWD, J5 LEFT OUTSIDE (REF) MIC, J6 LEFT IN-CUP (ERR) MIC, J7 TO RIGHT CUP, J8 LEFT SPEAKER, J9 BLE UART MODULE, Q1 AO3401A, Q2 MMBT3904, SW1 POWER, SW2 BOOT, U1 USBLC6-2SC6, U10 TPA6132A2, U2 MCP73831-2, U3 TPS63001, U4 LP5907-2.8, U5 STM32H743VIT6, U6 MCP6022, U7 MCP6022, U8 MCP6022, U9 MCP6022, Y1 25MHz

Commit message: main-board: routed except 11 connections; power tracks fit fine-pitch pads
- Power net class 0.40 -> 0.30 mm: a 0.4 mm track can't reach the 0.5 mm
  pitch pads of the LQFP-100, WQFN/QFN parts and USB-C at 0.18 mm
  clearance, so every power/GND pin of those parts was left unrouted
- tie_gnd_islands(): outer-layer GND pour islands without a via get one
  down to the inner plane (clearing other-net copper on every layer, no
  via-in-pad); islands too small for a via get a short fan-out track
- new stages: 'tie' (islands + refill + DRC on a finished board) and
  'complete' (one more autorouter round, then tie in a fresh process -
  works around KiCad 7 SWIG wrappers going stale after an SES import)

Result: 333 connections -> 11 unrouted (4 GND pads, AMP_INLN); no
clearance, short, drill or mask errors. Remaining DRC items are silk
cosmetics and library-table warnings.

Co-Authored-By: Claude Opus 5.5 <noreply@anthropic.com>
Claude-Session: https://claude.ai/code/session_011tw1Ap8ThDgVV2SB1vJK8Q
Parts:
- moved C15 32.7 mm to (110.1, 85.0), turned to 90 degrees
- moved TP8 29.7 mm to (126.3, 126.4)
- moved C44 26.7 mm to (110.3, 124.0), turned to -90 degrees
- moved C22 26.5 mm to (129.5, 124.8), turned to 0 degrees
- moved C14 24.1 mm to (121.8, 95.0), turned to 90 degrees
- moved C12 23.7 mm to (135.6, 114.6), turned to 180 degrees
- moved C11 23.1 mm to (131.7, 116.7), turned to 0 degrees
- moved C28 23.0 mm to (107.3, 119.2), turned to 180 degrees
- moved C23 20.6 mm to (107.7, 103.0), turned to 90 degrees
- moved C13 20.5 mm to (140.1, 97.8)
- moved C7 18.8 mm to (115.2, 105.2), turned to -90 degrees
- moved R22 17.5 mm to (115.1, 122.3), turned to 180 degrees
- moved C17 17.4 mm to (116.3, 99.9)
- moved C6 15.5 mm to (118.9, 96.6), turned to 180 degrees
- moved C16 12.8 mm to (116.1, 86.7)
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Routing:
- net 2V8A: track 0.00 -> 199.3 mm, vias 0 -> 10
- net 3V3: track 0.00 -> 181.6 mm, vias 0 -> 7
- net GND: track 0.00 -> 133.3 mm, vias 0 -> 70
- net VSYS: track 0.00 -> 97.9 mm, vias 0 -> 5
- net VMID: track 0.00 -> 57.0 mm, vias 0 -> 4
- net VBUS_F: track 0.00 -> 50.9 mm, vias 0 -> 2
- net ERR_L: track 0.00 -> 42.8 mm, vias 0 -> 4
- net VMID_DIV: track 0.00 -> 42.4 mm, vias 0 -> 2
- net VCAP: track 0.00 -> 38.3 mm, vias 0 -> 4
- net AMP_G1: track 0.00 -> 37.7 mm, vias 0 -> 2
- net BOOT0: track 0.00 -> 37.1 mm, vias 0 -> 2
- net BTN_HI: track 0.00 -> 36.3 mm, vias 0 -> 3
- net BLE_STATE: track 0.00 -> 35.3 mm, vias 0 -> 2
- net AMP_G0: track 0.00 -> 34.9 mm, vias 0 -> 2
- net REF_L: track 0.00 -> 34.8 mm, vias 0 -> 4
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- added copper zone on B.Cu, net GND
- added copper zone on F.Cu, net GND

Commit message: main-board: fully routed (0 unconnected), DRC clean, fab files
From 11 unrouted after Freerouting to 0, with hardware/gen/finish_route.py:
a grid A* router over F.Cu/In2.Cu/B.Cu that
- routes a boxed-in signal after ripping up the net that walls it in
  (AMP_INLN at U10.1; SPK_L re-routed at 0.2 mm - <= 56 mA peak)
- fans GND pads out to a via, an existing GND via or a tied GND pour
- rips up a whole wall net or only its segments near a pad, and saves only
  when every cut end re-joins
Also: tie stage always refills first; board min via 0.45/0.2 mm (JLCPCB
4-layer standard); documented .kicad_dru rules (GND through-holes solid to
the pour; one thermal spoke allowed on small GND pads); refs on F.Fab on
this dense board.

DRC: 0 unconnected, 0 clearance/short/hole/via/thermal errors. Left:
2 courtyard overlaps (J2/U2, J4/J1: bodies clear by 0.30 / 1.68 mm, the
overlap is the connectors' mating courtyard), 2 connector silk lines at
the board edge (clipped by the fab), library-table warnings (environment).
check_fit.py passes. Fab: gerbers + drill zip, JLC BOM + CPL, STEP, renders.

Co-Authored-By: Claude Opus 5.5 <noreply@anthropic.com>
Claude-Session: https://claude.ai/code/session_011tw1Ap8ThDgVV2SB1vJK8Q
Routing:
- net GND: track 133.3 -> 154.9 mm, vias 70 -> 83
- net VMID_DIV: track 42.4 -> 23.7 mm, vias 2 -> 3
- net SPK_L: track 19.4 -> 35.7 mm, vias 2 -> 4
- net DACL_OUT: track 25.4 -> 15.9 mm
- net AMP_INLN: track 0.00 -> 4.53 mm, vias 0 -> 2
- net BTN_B: track 19.9 -> 16.1 mm, vias 0 -> 4
- net DACL_B: track 7.06 -> 5.77 mm
- net 2V8A: track 199.3 -> 198.1 mm, vias 10 -> 12
- net DACR_A: track 15.1 -> 14.0 mm
- net ERRL_SKA: track 6.69 -> 6.06 mm
